Commit message: my algorithms

File: src/atom/urdf/atom.xacro (robot description, xacro)
@@ -241,5 +241,5 @@
 	<!-- Color of bot -->
 	<gazebo reference="left_wheel_front">
-		<material>Gazebo/Green</material>
+		<material>Gazebo/Black</material>
 		<kp>1000000.0</kp> <!-- kp and kd for rubber -->
 		<kd>100.0</kd>
@@ -250,5 +250,5 @@
 	</gazebo>
 	<gazebo reference="left_wheel_back">
-		<material>Gazebo/Green</material>
+		<material>Gazebo/Black</material>
 		<kp>1000000.0</kp> <!-- kp and kd for rubber -->
 		<kd>100.0</kd>
@@ -259,5 +259,5 @@
 	</gazebo>
 	<gazebo reference="right_wheel_front">
-		<material>Gazebo/Green</material>
+		<material>Gazebo/Black</material>
 		<kp>1000000.0</kp> <!-- kp and kd for rubber -->
 		<kd>100.0</kd>
@@ -268,5 +268,5 @@
 	</gazebo>
 	<gazebo reference="right_wheel_back">
-		<material>Gazebo/Green</material>
+		<material>Gazebo/Black</material>
 		<kp>1000000.0</kp> <!-- kp and kd for rubber -->
 		<kd>100.0</kd>
@@ -277,13 +277,44 @@
 	</gazebo>
 	<!--<gazebo reference="right_wheel">
-		<material>Gazebo/Green</material>
+		<material>Gazebo/Black</material>
 	</gazebo>-->
 	<gazebo reference="camera">
-		<material>Gazebo/Red</material>
+		<material>Gazebo/Orange</material>
 	</gazebo>
 	<gazebo reference="chassis">
-		<material>Gazebo/Blue</material>
+		<material>Gazebo/Yellow</material>
 	</gazebo>
 	<!-- Motor, Camera and Lidar Simulation -->
 	<xacro:include filename="$(find atom)/urdf/atom.gazebo" />
+	<gazebo reference="chassis">
+		<gravity>true</gravity>
+		<sensor name="imu_sensor" type="imu">
+     			<always_on>true</always_on>
+     			<update_rate>10</update_rate>
+     			<visualize>true</visualize>
+     			<topic>__default_topic__</topic>
+     			<plugin filename="libgazebo_ros_imu_sensor.so" name="imu_plugin">
+      				<topicName>imu</topicName>
+      				<bodyName>imu_link</bodyName>
+      				<updateRateHZ>10.0</updateRateHZ>
+      				<gaussianNoise>0.0</gaussianNoise>
+      				<xyzOffset>0 0 0</xyzOffset>
+      				<rpyOffset>0 0 -1.57</rpyOffset>
+      				<frameName>chassis</frameName>
+      				<initialOrientationAsReference>false</initialOrientationAsReference>
+     			</plugin>
+     			<pose>0 0 0 0 0 0</pose>
+    		</sensor>
+   	</gazebo>
+   	<gazebo>
+    		<plugin name="novatel_gps_sim" filename="libhector_gazebo_ros_gps.so">
+      			<alwaysOn>1</alwaysOn>
+      			<updateRate>10</updateRate>
+      			<bodyName>chassis</bodyName>
+      			<topicName>fix</topicName>
+      			<velocityTopicName>fix_velocity</velocityTopicName>
+      			<gaussianNoise>0.0 0.0 0.0</gaussianNoise>
+      			<velocityGaussianNoise>0.0 0.0 0.0</velocityGaussianNoise>
+    		</plugin>
+   	</gazebo>
 </robot>
